Commit message: Added missing prefix to base_footprint_joint

File: blue_description/xacro/bluerov2_heavy/urdf.xacro (robot description, xacro)
@@ -32,5 +32,5 @@
       </collision>
     </link>
-    <joint name="base_footprint_joint" type="fixed">
+    <joint name="${prefix}base_footprint_joint" type="fixed">
       <parent link="${prefix}base_footprint" />
       <child link="${prefix}base_link" />

File: blue_description/xacro/bluerov2_heavy_reach/urdf.xacro (robot description, xacro)
@@ -32,5 +32,5 @@
       </collision>
     </link>
-    <joint name="base_footprint_joint" type="fixed">
+    <joint name="${prefix}base_footprint_joint" type="fixed">
       <parent link="${prefix}base_footprint" />
       <child link="${prefix}base_link" />

Commit message: Integrate support for simulated camera (#73)
* Integrated camera and fixed camera localizer

* Fixed tf bugs

* precommit

* Added missing prefix to base_footprint_joint

* Cleaned up readme to discuss general framework instead of targeted framework

* Fixed readme grammar error

File: blue_description/xacro/bluerov2_heavy/urdf.xacro (robot description, xacro)
@@ -32,8 +32,13 @@
       </collision>
     </link>
-    <joint name="base_footprint_joint" type="fixed">
+    <joint name="${prefix}base_footprint_joint" type="fixed">
       <parent link="${prefix}base_footprint" />
       <child link="${prefix}base_link" />
     </joint>
+    <!-- Import camera macro -->
+    <xacro:include filename="$(find blue_description)/xacro/camera/urdf.xacro" />
+    <xacro:camera_urdf prefix="${prefix}" parent="${prefix}base_link">
+      <origin rpy="0 0 0" xyz="0.21 0 0.067" />
+    </xacro:camera_urdf>
     <!-- Import T200 macro -->
     <xacro:include filename="$(find blue_description)/xacro/t200/urdf.xacro" />

File: blue_description/xacro/bluerov2_heavy_reach/urdf.xacro (robot description, xacro)
@@ -32,8 +32,13 @@
       </collision>
     </link>
-    <joint name="base_footprint_joint" type="fixed">
+    <joint name="${prefix}base_footprint_joint" type="fixed">
       <parent link="${prefix}base_footprint" />
       <child link="${prefix}base_link" />
     </joint>
+    <!-- Import camera macro -->
+    <xacro:include filename="$(find blue_description)/xacro/camera/urdf.xacro" />
+    <xacro:camera_urdf prefix="${prefix}" parent="${prefix}base_link">
+      <origin rpy="0 0 0" xyz="0.21 0 0.067" />
+    </xacro:camera_urdf>
     <!-- Import T200 macro -->
     <xacro:include filename="$(find blue_description)/xacro/t200/urdf.xacro" />
