Commit message: Replaced package usage with find file in xacro

File: blue_description/xacro/bluerov2/urdf.xacro (robot description, xacro)
@@ -19,5 +19,5 @@
         <geometry>
           <mesh
-            filename="package://blue_description/meshes/bluerov2/bluerov2.dae"
+            filename="file://$(find blue_description)/meshes/bluerov2/bluerov2.dae"
             scale="0.025 0.025 0.025"
           />

File: blue_description/xacro/bluerov2_heavy/urdf.xacro (robot description, xacro)
@@ -19,5 +19,5 @@
         <geometry>
           <mesh
-            filename="package://blue_description/meshes/bluerov2_heavy/bluerov2_heavy.dae"
+            filename="file://$(find blue_description)/meshes/bluerov2_heavy/bluerov2_heavy.dae"
             scale="0.025 0.025 0.025"
           />

File: blue_description/xacro/bluerov2_heavy_reach/urdf.xacro (robot description, xacro)
@@ -19,5 +19,5 @@
         <geometry>
           <mesh
-            filename="package://blue_description/meshes/bluerov2_heavy_reach/bluerov2_heavy_reach.dae"
+            filename="file://$(find blue_description)/meshes/bluerov2_heavy_reach/bluerov2_heavy_reach.dae"
             scale="0.025 0.025 0.025"
           />

File: blue_description/xacro/t200/urdf.xacro (robot description, xacro)
@@ -17,10 +17,10 @@
         <xacro:if value="${ccw}">
           <geometry>
-            <mesh filename="package://blue_description/meshes/t200/ccw_prop.dae" />
+            <mesh filename="file://$(find blue_description)/meshes/t200/ccw_prop.dae" />
           </geometry>
         </xacro:if>
         <xacro:unless value="${ccw}">
           <geometry>
-            <mesh filename="package://blue_description/meshes/t200/cw_prop.dae" />
+            <mesh filename="file://$(find blue_description)/meshes/t200/cw_prop.dae" />
           </geometry>
         </xacro:unless>

Commit message: Fixed camera frame

File: blue_description/xacro/bluerov2/urdf.xacro (robot description, xacro)
@@ -39,5 +39,5 @@
     <xacro:include filename="$(find blue_description)/xacro/camera/urdf.xacro" />
     <xacro:camera_urdf prefix="${prefix}" parent="${prefix}base_link">
-      <origin rpy="0 0 0" xyz="0.21 0 0.067" />
+      <origin rpy="-1.571 0 -1.571" xyz="0.21 0 0.067" />
     </xacro:camera_urdf>
     <!-- Import T200 macro -->

File: blue_description/xacro/bluerov2_heavy/urdf.xacro (robot description, xacro)
@@ -39,5 +39,5 @@
     <xacro:include filename="$(find blue_description)/xacro/camera/urdf.xacro" />
     <xacro:camera_urdf prefix="${prefix}" parent="${prefix}base_link">
-      <origin rpy="0 0 0" xyz="0.21 0 0.067" />
+      <origin rpy="-1.571 0 -1.571" xyz="0.21 0 0.067" />
     </xacro:camera_urdf>
     <!-- Import T200 macro -->

File: blue_description/xacro/bluerov2_heavy_reach/urdf.xacro (robot description, xacro)
@@ -39,5 +39,5 @@
     <xacro:include filename="$(find blue_description)/xacro/camera/urdf.xacro" />
     <xacro:camera_urdf prefix="${prefix}" parent="${prefix}base_link">
-      <origin rpy="0 0 0" xyz="0.21 0 0.067" />
+      <origin rpy="-1.571 0 -1.571" xyz="0.21 0 0.067" />
     </xacro:camera_urdf>
     <!-- Import T200 macro -->
