Commit message: Clearly hotfixes were a bad idea

File: blue_description/xacro/bluerov2/gazebo.xacro (robot description, xacro)
@@ -2,4 +2,5 @@
 <robot xmlns:xacro="http://ros.org/wiki/xacro">
   <xacro:macro name="bluerov2_gazebo" params="prefix">
+    <xacro:property name="model" value="bluerov2" />
     <gazebo>
       <plugin name="ArduPilotPlugin" filename="libArduPilotPlugin.so">
@@ -22,5 +23,5 @@
           <servo_max>1900</servo_max>
           <type>COMMAND</type>
-          <cmd_topic>/model/blue/joint/${prefix}thruster1_joint/cmd_thrust</cmd_topic>
+          <cmd_topic>/model/${model}/joint/${prefix}thruster1_joint/cmd_thrust</cmd_topic>
           <offset>-0.5</offset>
           <multiplier>100</multiplier>
@@ -31,5 +32,5 @@
           <servo_max>1900</servo_max>
           <type>COMMAND</type>
-          <cmd_topic>/model/blue/joint/${prefix}thruster2_joint/cmd_thrust</cmd_topic>
+          <cmd_topic>/model/${model}/joint/${prefix}thruster2_joint/cmd_thrust</cmd_topic>
           <offset>-0.5</offset>
           <multiplier>100</multiplier>
@@ -40,5 +41,5 @@
           <servo_max>1900</servo_max>
           <type>COMMAND</type>
-          <cmd_topic>/model/blue/joint/${prefix}thruster3_joint/cmd_thrust</cmd_topic>
+          <cmd_topic>/model/${model}/joint/${prefix}thruster3_joint/cmd_thrust</cmd_topic>
           <offset>-0.5</offset>
           <multiplier>100</multiplier>
@@ -49,5 +50,5 @@
           <servo_max>1900</servo_max>
           <type>COMMAND</type>
-          <cmd_topic>/model/blue/joint/${prefix}thruster4_joint/cmd_thrust</cmd_topic>
+          <cmd_topic>/model/${model}/joint/${prefix}thruster4_joint/cmd_thrust</cmd_topic>
           <offset>-0.5</offset>
           <multiplier>100</multiplier>
@@ -58,5 +59,5 @@
           <servo_max>1900</servo_max>
           <type>COMMAND</type>
-          <cmd_topic>/model/blue/joint/${prefix}thruster5_joint/cmd_thrust</cmd_topic>
+          <cmd_topic>/model/${model}/joint/${prefix}thruster5_joint/cmd_thrust</cmd_topic>
           <offset>-0.5</offset>
           <multiplier>100</multiplier>
@@ -67,5 +68,5 @@
           <servo_max>1900</servo_max>
           <type>COMMAND</type>
-          <cmd_topic>/model/blue/joint/${prefix}thruster6_joint/cmd_thrust</cmd_topic>
+          <cmd_topic>/model/${model}/joint/${prefix}thruster6_joint/cmd_thrust</cmd_topic>
           <offset>-0.5</offset>
           <multiplier>100</multiplier>
@@ -122,10 +123,10 @@
     <!-- Include the T200 Gazebo macro -->
     <xacro:include filename="$(find blue_description)/xacro/t200/gazebo.xacro" />
-    <xacro:t200_gazebo namespace="bluerov2" prefix="${prefix}" id="1" ccw="true" />
-    <xacro:t200_gazebo namespace="bluerov2" prefix="${prefix}" id="2" ccw="true" />
-    <xacro:t200_gazebo namespace="bluerov2" prefix="${prefix}" id="3" />
-    <xacro:t200_gazebo namespace="bluerov2" prefix="${prefix}" id="4" />
-    <xacro:t200_gazebo namespace="bluerov2" prefix="${prefix}" id="5" ccw="true" />
-    <xacro:t200_gazebo namespace="bluerov2" prefix="${prefix}" id="6" />
+    <xacro:t200_gazebo namespace="${model}" prefix="${prefix}" id="1" ccw="true" />
+    <xacro:t200_gazebo namespace="${model}" prefix="${prefix}" id="2" ccw="true" />
+    <xacro:t200_gazebo namespace="${model}" prefix="${prefix}" id="3" />
+    <xacro:t200_gazebo namespace="${model}" prefix="${prefix}" id="4" />
+    <xacro:t200_gazebo namespace="${model}" prefix="${prefix}" id="5" ccw="true" />
+    <xacro:t200_gazebo namespace="${model}" prefix="${prefix}" id="6" />
   </xacro:macro>
 </robot>

File: blue_description/xacro/bluerov2_heavy/gazebo.xacro (robot description, xacro)
@@ -2,4 +2,5 @@
 <robot xmlns:xacro="http://ros.org/wiki/xacro">
   <xacro:macro name="bluerov2_heavy_gazebo" params="prefix">
+    <xacro:property name="model" value="bluerov2_heavy" />
     <gazebo>
       <plugin name="ArduPilotPlugin" filename="libArduPilotPlugin.so">
@@ -22,5 +23,5 @@
           <servo_max>1900</servo_max>
           <type>COMMAND</type>
-          <cmd_topic>/model/blue/joint/${prefix}thruster1_joint/cmd_thrust</cmd_topic>
+          <cmd_topic>/model/${model}/joint/${prefix}thruster1_joint/cmd_thrust</cmd_topic>
           <offset>-0.5</offset>
           <multiplier>100</multiplier>
@@ -31,5 +32,5 @@
           <servo_max>1900</servo_max>
           <type>COMMAND</type>
-          <cmd_topic>/model/blue/joint/${prefix}thruster2_joint/cmd_thrust</cmd_topic>
+          <cmd_topic>/model/${model}/joint/${prefix}thruster2_joint/cmd_thrust</cmd_topic>
           <offset>-0.5</offset>
           <multiplier>100</multiplier>
@@ -40,5 +41,5 @@
           <servo_max>1900</servo_max>
           <type>COMMAND</type>
-          <cmd_topic>/model/blue/joint/${prefix}thruster3_joint/cmd_thrust</cmd_topic>
+          <cmd_topic>/model/${model}/joint/${prefix}thruster3_joint/cmd_thrust</cmd_topic>
           <offset>-0.5</offset>
           <multiplier>100</multiplier>
@@ -49,5 +50,5 @@
           <servo_max>1900</servo_max>
           <type>COMMAND</type>
-          <cmd_topic>/model/blue/joint/${prefix}thruster4_joint/cmd_thrust</cmd_topic>
+          <cmd_topic>/model/${model}/joint/${prefix}thruster4_joint/cmd_thrust</cmd_topic>
           <offset>-0.5</offset>
           <multiplier>100</multiplier>
@@ -58,5 +59,5 @@
           <servo_max>1900</servo_max>
           <type>COMMAND</type>
-          <cmd_topic>/model/blue/joint/${prefix}thruster5_joint/cmd_thrust</cmd_topic>
+          <cmd_topic>/model/${model}/joint/${prefix}thruster5_joint/cmd_thrust</cmd_topic>
           <offset>-0.5</offset>
           <multiplier>100</multiplier>
@@ -67,5 +68,5 @@
           <servo_max>1900</servo_max>
           <type>COMMAND</type>
-          <cmd_topic>/model/blue/joint/${prefix}thruster6_joint/cmd_thrust</cmd_topic>
+          <cmd_topic>/model/${model}/joint/${prefix}thruster6_joint/cmd_thrust</cmd_topic>
           <offset>-0.5</offset>
           <multiplier>100</multiplier>
@@ -76,5 +77,5 @@
           <servo_max>1900</servo_max>
           <type>COMMAND</type>
-          <cmd_topic>/model/blue/joint/${prefix}thruster7_joint/cmd_thrust</cmd_topic>
+          <cmd_topic>/model/${model}/joint/${prefix}thruster7_joint/cmd_thrust</cmd_topic>
           <offset>-0.5</offset>
           <multiplier>100</multiplier>
@@ -85,5 +86,5 @@
           <servo_max>1900</servo_max>
           <type>COMMAND</type>
-          <cmd_topic>/model/blue/joint/${prefix}thruster8_joint/cmd_thrust</cmd_topic>
+          <cmd_topic>/model/${model}/joint/${prefix}thruster8_joint/cmd_thrust</cmd_topic>
           <offset>-0.5</offset>
           <multiplier>100</multiplier>
@@ -140,12 +141,12 @@
     <!-- Include the T200 Gazebo macro -->
     <xacro:include filename="$(find blue_description)/xacro/t200/gazebo.xacro" />
-    <xacro:t200_gazebo namespace="bluerov2_heavy" prefix="${prefix}" id="1" ccw="true" />
-    <xacro:t200_gazebo namespace="bluerov2_heavy" prefix="${prefix}" id="2" ccw="true" />
-    <xacro:t200_gazebo namespace="bluerov2_heavy" prefix="${prefix}" id="3" />
-    <xacro:t200_gazebo namespace="bluerov2_heavy" prefix="${prefix}" id="4" />
-    <xacro:t200_gazebo namespace="bluerov2_heavy" prefix="${prefix}" id="5" ccw="true" />
-    <xacro:t200_gazebo namespace="bluerov2_heavy" prefix="${prefix}" id="6" />
-    <xacro:t200_gazebo namespace="bluerov2_heavy" prefix="${prefix}" id="7" />
-    <xacro:t200_gazebo namespace="bluerov2_heavy" prefix="${prefix}" id="8" ccw="true" />
+    <xacro:t200_gazebo namespace="${model}" prefix="${prefix}" id="1" ccw="true" />
+    <xacro:t200_gazebo namespace="${model}" prefix="${prefix}" id="2" ccw="true" />
+    <xacro:t200_gazebo namespace="${model}" prefix="${prefix}" id="3" />
+    <xacro:t200_gazebo namespace="${model}" prefix="${prefix}" id="4" />
+    <xacro:t200_gazebo namespace="${model}" prefix="${prefix}" id="5" ccw="true" />
+    <xacro:t200_gazebo namespace="${model}" prefix="${prefix}" id="6" />
+    <xacro:t200_gazebo namespace="${model}" prefix="${prefix}" id="7" />
+    <xacro:t200_gazebo namespace="${model}" prefix="${prefix}" id="8" ccw="true" />
   </xacro:macro>
 </robot>

File: blue_description/xacro/bluerov2_heavy_reach/gazebo.xacro (robot description, xacro)
@@ -2,4 +2,5 @@
 <robot xmlns:xacro="http://ros.org/wiki/xacro">
   <xacro:macro name="bluerov2_heavy_reach_gazebo" params="prefix">
+    <xacro:property name="model" value="bluerov2_heavy_reach" />
     <gazebo>
       <plugin name="ArduPilotPlugin" filename="libArduPilotPlugin.so">
@@ -22,5 +23,5 @@
           <servo_max>1900</servo_max>
           <type>COMMAND</type>
-          <cmd_topic>/model/blue/joint/${prefix}thruster1_joint/cmd_thrust</cmd_topic>
+          <cmd_topic>/model/${model}/joint/${prefix}thruster1_joint/cmd_thrust</cmd_topic>
           <offset>-0.5</offset>
           <multiplier>100</multiplier>
@@ -31,5 +32,5 @@
           <servo_max>1900</servo_max>
           <type>COMMAND</type>
-          <cmd_topic>/model/blue/joint/${prefix}thruster2_joint/cmd_thrust</cmd_topic>
+          <cmd_topic>/model/${model}/joint/${prefix}thruster2_joint/cmd_thrust</cmd_topic>
           <offset>-0.5</offset>
           <multiplier>100</multiplier>
@@ -40,5 +41,5 @@
           <servo_max>1900</servo_max>
           <type>COMMAND</type>
-          <cmd_topic>/model/blue/joint/${prefix}thruster3_joint/cmd_thrust</cmd_topic>
+          <cmd_topic>/model/${model}/joint/${prefix}thruster3_joint/cmd_thrust</cmd_topic>
           <offset>-0.5</offset>
           <multiplier>100</multiplier>
@@ -49,5 +50,5 @@
           <servo_max>1900</servo_max>
           <type>COMMAND</type>
-          <cmd_topic>/model/blue/joint/${prefix}thruster4_joint/cmd_thrust</cmd_topic>
+          <cmd_topic>/model/${model}/joint/${prefix}thruster4_joint/cmd_thrust</cmd_topic>
           <offset>-0.5</offset>
           <multiplier>100</multiplier>
@@ -58,5 +59,5 @@
           <servo_max>1900</servo_max>
           <type>COMMAND</type>
-          <cmd_topic>/model/blue/joint/${prefix}thruster5_joint/cmd_thrust</cmd_topic>
+          <cmd_topic>/model/${model}/joint/${prefix}thruster5_joint/cmd_thrust</cmd_topic>
           <offset>-0.5</offset>
           <multiplier>100</multiplier>
@@ -67,5 +68,5 @@
           <servo_max>1900</servo_max>
           <type>COMMAND</type>
-          <cmd_topic>/model/blue/joint/${prefix}thruster6_joint/cmd_thrust</cmd_topic>
+          <cmd_topic>/model/${model}/joint/${prefix}thruster6_joint/cmd_thrust</cmd_topic>
           <offset>-0.5</offset>
           <multiplier>100</multiplier>
@@ -76,5 +77,5 @@
           <servo_max>1900</servo_max>
           <type>COMMAND</type>
-          <cmd_topic>/model/blue/joint/${prefix}thruster7_joint/cmd_thrust</cmd_topic>
+          <cmd_topic>/model/${model}/joint/${prefix}thruster7_joint/cmd_thrust</cmd_topic>
           <offset>-0.5</offset>
           <multiplier>100</multiplier>
@@ -85,5 +86,5 @@
           <servo_max>1900</servo_max>
           <type>COMMAND</type>
-          <cmd_topic>/model/blue/joint/${prefix}thruster8_joint/cmd_thrust</cmd_topic>
+          <cmd_topic>/model/${model}/joint/${prefix}thruster8_joint/cmd_thrust</cmd_topic>
           <offset>-0.5</offset>
           <multiplier>100</multiplier>
@@ -140,12 +141,12 @@
     <!-- Include the T200 Gazebo macro -->
     <xacro:include filename="$(find blue_description)/xacro/t200/gazebo.xacro" />
-    <xacro:t200_gazebo namespace="bluerov2_heavy_reach" prefix="${prefix}" id="1" ccw="true" />
-    <xacro:t200_gazebo namespace="bluerov2_heavy_reach" prefix="${prefix}" id="2" ccw="true" />
-    <xacro:t200_gazebo namespace="bluerov2_heavy_reach" prefix="${prefix}" id="3" />
-    <xacro:t200_gazebo namespace="bluerov2_heavy_reach" prefix="${prefix}" id="4" />
-    <xacro:t200_gazebo namespace="bluerov2_heavy_reach" prefix="${prefix}" id="5" ccw="true" />
-    <xacro:t200_gazebo namespace="bluerov2_heavy_reach" prefix="${prefix}" id="6" />
-    <xacro:t200_gazebo namespace="bluerov2_heavy_reach" prefix="${prefix}" id="7" />
-    <xacro:t200_gazebo namespace="bluerov2_heavy_reach" prefix="${prefix}" id="8" ccw="true" />
+    <xacro:t200_gazebo namespace="${model}" prefix="${prefix}" id="1" ccw="true" />
+    <xacro:t200_gazebo namespace="${model}" prefix="${prefix}" id="2" ccw="true" />
+    <xacro:t200_gazebo namespace="${model}" prefix="${prefix}" id="3" />
+    <xacro:t200_gazebo namespace="${model}" prefix="${prefix}" id="4" />
+    <xacro:t200_gazebo namespace="${model}" prefix="${prefix}" id="5" ccw="true" />
+    <xacro:t200_gazebo namespace="${model}" prefix="${prefix}" id="6" />
+    <xacro:t200_gazebo namespace="${model}" prefix="${prefix}" id="7" />
+    <xacro:t200_gazebo namespace="${model}" prefix="${prefix}" id="8" ccw="true" />
   </xacro:macro>
 </robot>

Commit message: Fixed bugs in joy integration and camera frames

File: blue_description/xacro/bluerov2/gazebo.xacro (robot description, xacro)
@@ -123,5 +123,5 @@
     <!-- Include the camera Gazebo macro -->
     <xacro:include filename="$(find blue_description)/xacro/camera/gazebo.xacro" />
-    <xacro:camera_gazebo reference="${prefix}camera_link" />
+    <xacro:camera_gazebo reference="${prefix}camera_mount_link" />
     <!-- Include the T200 Gazebo macro -->
     <xacro:include filename="$(find blue_description)/xacro/t200/gazebo.xacro" />

File: blue_description/xacro/bluerov2/urdf.xacro (robot description, xacro)
@@ -39,5 +39,5 @@
     <xacro:include filename="$(find blue_description)/xacro/camera/urdf.xacro" />
     <xacro:camera_urdf prefix="${prefix}" parent="${prefix}base_link">
-      <origin rpy="-1.571 0 -1.571" xyz="0.21 0 0.067" />
+      <origin rpy="0 0 0" xyz="0.21 0 0.067" />
     </xacro:camera_urdf>
     <!-- Import T200 macro -->

File: blue_description/xacro/bluerov2_heavy/gazebo.xacro (robot description, xacro)
@@ -141,5 +141,5 @@
     <!-- Include the camera Gazebo macro -->
     <xacro:include filename="$(find blue_description)/xacro/camera/gazebo.xacro" />
-    <xacro:camera_gazebo reference="${prefix}camera_link" />
+    <xacro:camera_gazebo reference="${prefix}camera_mount_link" />
     <!-- Include the T200 Gazebo macro -->
     <xacro:include filename="$(find blue_description)/xacro/t200/gazebo.xacro" />

File: blue_description/xacro/bluerov2_heavy/urdf.xacro (robot description, xacro)
@@ -39,5 +39,5 @@
     <xacro:include filename="$(find blue_description)/xacro/camera/urdf.xacro" />
     <xacro:camera_urdf prefix="${prefix}" parent="${prefix}base_link">
-      <origin rpy="-1.571 0 -1.571" xyz="0.21 0 0.067" />
+      <origin rpy="0 0 0" xyz="0.21 0 0.067" />
     </xacro:camera_urdf>
     <!-- Import T200 macro -->

File: blue_description/xacro/bluerov2_heavy_reach/gazebo.xacro (robot description, xacro)
@@ -141,5 +141,5 @@
     <!-- Include the camera Gazebo macro -->
     <xacro:include filename="$(find blue_description)/xacro/camera/gazebo.xacro" />
-    <xacro:camera_gazebo reference="${prefix}camera_link" />
+    <xacro:camera_gazebo reference="${prefix}camera_mount_link" />
     <!-- Include the T200 Gazebo macro -->
     <xacro:include filename="$(find blue_description)/xacro/t200/gazebo.xacro" />

File: blue_description/xacro/bluerov2_heavy_reach/urdf.xacro (robot description, xacro)
@@ -39,5 +39,5 @@
     <xacro:include filename="$(find blue_description)/xacro/camera/urdf.xacro" />
     <xacro:camera_urdf prefix="${prefix}" parent="${prefix}base_link">
-      <origin rpy="-1.571 0 -1.571" xyz="0.21 0 0.067" />
+      <origin rpy="0 0 0" xyz="0.21 0 0.067" />
     </xacro:camera_urdf>
     <!-- Import T200 macro -->

File: blue_description/xacro/camera/urdf.xacro (robot description, xacro)
@@ -15,7 +15,25 @@
       </inertial>
     </link>
-    <joint name="${prefix}camera_joint" type="fixed">
+    <link name="${prefix}camera_mount_link">
+      <inertial>
+        <mass value="0.0001" />
+        <inertia
+          ixx="0.0001"
+          ixy="0"
+          ixz="0"
+          iyy="0.0001"
+          iyz="0"
+          izz="0.0001"
+        />
+      </inertial>
+    </link>
+    <joint name="${prefix}camera_mount_joint" type="fixed">
       <xacro:insert_block name="origin" />
       <parent link="${parent}" />
+      <child link="${prefix}camera_mount_link" />
+    </joint>
+    <joint name="${prefix}camera_joint" type="fixed">
+      <origin rpy="-1.571 0 -1.571" xyz="0 0 0" />
+      <parent link="${prefix}camera_mount_link" />
       <child link="${prefix}camera_link" />
     </joint>
