Commit message: compatible with prefixes and namespaces

File: blue_demos/control_integration/description/ros2_control/bluerov2_heavy.ros2_control.xacro (robot description, xacro)
@@ -1,10 +1,11 @@
 <?xml version="1.0"?>
 <robot xmlns:xacro="http://www.ros.org/wiki/xacro">
-  <xacro:macro name="ardusub_thruster_system" params="prefix name max_set_param_attempts:=^3">
+  <xacro:macro name="ardusub_thruster_system"
+    params="prefix name use_mavros_odom mavros_odom_topic max_set_param_attempts:=^3">
     <ros2_control name="${name}" type="system">
       <hardware>
         <plugin>thruster_hardware/ThrusterHardware</plugin>
         <param name="max_set_param_attempts">${max_set_param_attempts}</param>
-        <param name="is_odom_si_present">true</param>
+        <param name="namespace">${prefix}</param>
       </hardware>
       <joint name="${prefix}thruster1_joint">
@@ -57,4 +58,14 @@
       </joint>
     </ros2_control>
+    <xacro:if value="${use_mavros_odom}">
+      <ros2_control name="MavrosOdomSensor" type="sensor">
+        <hardware>
+          <plugin>mavros_odom_sensor/MavrosOdomSensor</plugin>
+          <param name="max_set_param_attempts">${max_set_param_attempts}</param>
+          <param name="mavros_odom_topic">${mavros_odom_topic}</param>
+          <param name="namespace">${prefix}</param>
+        </hardware>
+      </ros2_control>
+    </xacro:if>
   </xacro:macro>
 </robot>

File: blue_demos/control_integration/description/urdf/bluerov2_heavy.config.xacro (robot description, xacro)
@@ -3,4 +3,8 @@
   <xacro:arg name="prefix" default="" />
   <xacro:arg name="use_sim" default="false" />
+  <xacro:arg name="fdm_port_in" default="9002" />
+  <xacro:arg name="fdm_port_out" default="9003" />
+  <xacro:arg name="use_mavros_odom" default="false" />
+  <xacro:arg name="mavros_odom_topic" default="/mavros/local_position/odom" />
   <!-- Import BlueROV2 macro -->
   <xacro:include filename="$(find blue_description)/description/bluerov2_heavy/urdf.xacro" />
@@ -9,9 +13,13 @@
   <xacro:if value="$(arg use_sim)">
     <xacro:include filename="$(find blue_description)/description/bluerov2_heavy/gazebo.xacro" />
-    <xacro:bluerov2_heavy_gazebo prefix="$(arg prefix)" />
+    <xacro:bluerov2_heavy_gazebo prefix="$(arg prefix)" fdm_port_in="$(arg fdm_port_in)"
+      fdm_port_out="$(arg fdm_port_out)" />
   </xacro:if>
   <!-- Import ros2_control macro -->
   <xacro:include
-    filename="$(find blue_demos)/control_integration/description/ros2_control/bluerov2_heavy.ros2_control.xacro" />
-  <xacro:ardusub_thruster_system prefix="$(arg prefix)" name="$(arg prefix)bluerov2_heavy_thrusters" />
+    filename="$(find
+  blue_demos)/control_integration/description/ros2_control/bluerov2_heavy.ros2_control.xacro" />
+  <xacro:ardusub_thruster_system prefix="$(arg prefix)" use_mavros_odom="$(arg use_mavros_odom)"
+    mavros_odom_topic="$(arg mavros_odom_topic)" name="$(arg prefix)bluerov2_heavy_thrusters"
+  />
 </robot>

File: blue_description/description/bluerov2_heavy/gazebo.xacro (robot description, xacro)
@@ -1,10 +1,11 @@
 <?xml version="1.0"?>
 <robot xmlns:xacro="http://ros.org/wiki/xacro">
-  <xacro:macro name="bluerov2_heavy_gazebo" params="prefix">
+  <xacro:macro name="bluerov2_heavy_gazebo" params="prefix fdm_port_in fdm_port_out">
     <xacro:property name="model" value="${prefix}bluerov2_heavy" />
     <gazebo>
       <plugin name="ArduPilotPlugin" filename="libArduPilotPlugin.so">
         <fdm_addr>127.0.0.1</fdm_addr>
-        <fdm_port_in>9002</fdm_port_in>
+        <fdm_port_in>${fdm_port_in}</fdm_port_in>
+        <fdm_port_out>${fdm_port_out}</fdm_port_out>
         <connectionTimeoutMaxCount>5</connectionTimeoutMaxCount>
         <lock_step>1</lock_step>

File: blue_description/description/camera/gazebo.xacro (robot description, xacro)
@@ -3,5 +3,5 @@
   <xacro:macro name="camera_gazebo" params="reference prefix">
     <!-- Camera sensors plugin -->
-    <gazebo>
+    <!-- <gazebo>
       <plugin
         filename="gz-sim-sensors-system"
@@ -9,5 +9,5 @@
         <render_engine>ogre2</render_engine>
       </plugin>
-    </gazebo>
+    </gazebo> -->
     <!-- Camera sensor -->
     <gazebo reference="${reference}">
