Commit message: use updated auv_controllers api

File: blue_demos/control_integration/description/ros2_control/bluerov2.ros2_control.xacro (robot description, xacro)
@@ -51,4 +51,15 @@
       </hardware>
     </ros2_control>
+    <hydrodynamics>
+      <mass>10.0</mass>
+      <inertia ixx="0.16" iyy="0.16" izz="0.16" />
+      <added_mass Xdu="-5.50" Ydv="-12.70" Zdw="-14.60" Kdp="-0.12" Mdq="-0.12" Ndr="-0.12" />
+      <linear_damping Xu="-4.03" Yv="-6.22" Zw="-5.18" Kp="-0.07" Mq="-0.07" Nr="-0.07" />
+      <quadratic_damping Xuu="-18.18" Yvv="-21.66" Zww="-36.99" Kpp="-1.55" Mqq="-1.55" Nrr="-1.55" />
+      <weight>98.1</weight>
+      <buoyancy>100.06</buoyancy>
+      <center_of_gravity x="0.0" y="0.0" z="0.0" />
+      <center_of_buoyancy x="0.0" y="0.0" z="0.0" />
+    </hydrodynamics>
   </xacro:macro>
 </robot>

File: blue_demos/control_integration/description/ros2_control/bluerov2_heavy.ros2_control.xacro (robot description, xacro)
@@ -56,4 +56,22 @@
       </joint>
     </ros2_control>
+    <ros2_control name="${name}_odom_sensor" type="sensor">
+      <hardware>
+        <plugin>topic_sensors/OdomSensor</plugin>
+        <param name="topic">/model/bluerov2/odometry_fsd</param>
+        <param name="prefix">${prefix}</param>
+      </hardware>
+    </ros2_control>
+    <hydrodynamics>
+      <mass>13.5</mass>
+      <inertia ixx="0.16" iyy="0.16" izz="0.16" />
+      <added_mass Xdu="-5.50" Ydv="-12.70" Zdw="-14.60" Kdp="-0.12" Mdq="-0.12" Ndr="-0.12" />
+      <linear_damping Xu="-4.03" Yv="-6.22" Zw="-5.18" Kp="-0.07" Mq="-0.07" Nr="-0.07" />
+      <quadratic_damping Xuu="-18.18" Yvv="-21.66" Zww="-36.99" Kpp="-1.55" Mqq="-1.55" Nrr="-1.55" />
+      <weight>98.1</weight>
+      <buoyancy>112.80</buoyancy>
+      <center_of_gravity x="0.0" y="0.0" z="0.0" />
+      <center_of_buoyancy x="0.0" y="0.0" z="0.0" />
+    </hydrodynamics>
   </xacro:macro>
 </robot>

Commit message: continue porting angler to blue

File: blue_demos/control_integration/description/ros2_control/bluerov2.ros2_control.xacro (robot description, xacro)
@@ -51,15 +51,4 @@
       </hardware>
     </ros2_control>
-    <hydrodynamics>
-      <mass>10.0</mass>
-      <inertia ixx="0.16" iyy="0.16" izz="0.16" />
-      <added_mass Xdu="-5.50" Ydv="-12.70" Zdw="-14.60" Kdp="-0.12" Mdq="-0.12" Ndr="-0.12" />
-      <linear_damping Xu="-4.03" Yv="-6.22" Zw="-5.18" Kp="-0.07" Mq="-0.07" Nr="-0.07" />
-      <quadratic_damping Xuu="-18.18" Yvv="-21.66" Zww="-36.99" Kpp="-1.55" Mqq="-1.55" Nrr="-1.55" />
-      <weight>98.1</weight>
-      <buoyancy>100.06</buoyancy>
-      <center_of_gravity x="0.0" y="0.0" z="0.0" />
-      <center_of_buoyancy x="0.0" y="0.0" z="0.0" />
-    </hydrodynamics>
   </xacro:macro>
 </robot>

File: blue_demos/control_integration/description/ros2_control/bluerov2_heavy.ros2_control.xacro (robot description, xacro)
@@ -63,15 +63,4 @@
       </hardware>
     </ros2_control>
-    <hydrodynamics>
-      <mass>13.5</mass>
-      <inertia ixx="0.16" iyy="0.16" izz="0.16" />
-      <added_mass Xdu="-5.50" Ydv="-12.70" Zdw="-14.60" Kdp="-0.12" Mdq="-0.12" Ndr="-0.12" />
-      <linear_damping Xu="-4.03" Yv="-6.22" Zw="-5.18" Kp="-0.07" Mq="-0.07" Nr="-0.07" />
-      <quadratic_damping Xuu="-18.18" Yvv="-21.66" Zww="-36.99" Kpp="-1.55" Mqq="-1.55" Nrr="-1.55" />
-      <weight>98.1</weight>
-      <buoyancy>112.80</buoyancy>
-      <center_of_gravity x="0.0" y="0.0" z="0.0" />
-      <center_of_buoyancy x="0.0" y="0.0" z="0.0" />
-    </hydrodynamics>
   </xacro:macro>
 </robot>

File: blue_demos/control_integration/description/urdf/bluerov2.config.xacro (robot description, xacro)
@@ -1,17 +1,15 @@
 <?xml version="1.0"?>
 <robot name="bluerov2" xmlns:xacro="http://ros.org/wiki/xacro">
+  <xacro:include filename="$(find blue_description)/description/bluerov2/urdf.xacro" />
+  <xacro:include filename="$(find blue_description)/description/bluerov2/gazebo.xacro" />
+  <xacro:include filename="$(find blue_demos)/control_integration/description/ros2_control/bluerov2.ros2_control.xacro" />
+  <xacro:include filename="$(find blue_demos)/control_integration/description/ros2_control/bluerov2.model.xacro" />
   <xacro:arg name="prefix" default="" />
   <xacro:arg name="use_sim" default="false" />
-  <!-- Import BlueROV2 macro -->
-  <xacro:include filename="$(find blue_description)/description/bluerov2/urdf.xacro" />
   <xacro:bluerov2_urdf prefix="$(arg prefix)" />
-  <!-- Import the Gazebo macro -->
   <xacro:if value="$(arg use_sim)">
-    <xacro:include filename="$(find blue_description)/description/bluerov2/gazebo.xacro" />
     <xacro:bluerov2_gazebo prefix="$(arg prefix)" />
   </xacro:if>
-  <!-- Import ros2_control macro -->
-  <xacro:include
-    filename="$(find blue_demos)/control_integration/description/ros2_control/bluerov2.ros2_control.xacro" />
+  <xacro:bluerov2_model />
   <xacro:ardusub_thruster_system prefix="$(arg prefix)" name="bluerov2_thrusters" />
 </robot>

File: blue_demos/control_integration/description/urdf/bluerov2_heavy.config.xacro (robot description, xacro)
@@ -1,17 +1,15 @@
 <?xml version="1.0"?>
 <robot name="bluerov2_heavy" xmlns:xacro="http://ros.org/wiki/xacro">
+  <xacro:include filename="$(find blue_description)/description/bluerov2_heavy/urdf.xacro" />
+  <xacro:include filename="$(find blue_description)/description/bluerov2_heavy/gazebo.xacro" />
+  <xacro:include filename="$(find blue_demos)/control_integration/description/ros2_control/bluerov2_heavy.ros2_control.xacro" />
+  <xacro:include filename="$(find blue_demos)/control_integration/description/ros2_control/bluerov2.model.xacro" />
   <xacro:arg name="prefix" default="" />
   <xacro:arg name="use_sim" default="false" />
-  <!-- Import BlueROV2 macro -->
-  <xacro:include filename="$(find blue_description)/description/bluerov2_heavy/urdf.xacro" />
   <xacro:bluerov2_heavy_urdf prefix="$(arg prefix)" />
-  <!-- Import the Gazebo macro -->
   <xacro:if value="$(arg use_sim)">
-    <xacro:include filename="$(find blue_description)/description/bluerov2_heavy/gazebo.xacro" />
     <xacro:bluerov2_heavy_gazebo prefix="$(arg prefix)" />
   </xacro:if>
-  <!-- Import ros2_control macro -->
-  <xacro:include
-    filename="$(find blue_demos)/control_integration/description/ros2_control/bluerov2_heavy.ros2_control.xacro" />
+  <xacro:bluerov2_heavy_model />
   <xacro:ardusub_thruster_system prefix="$(arg prefix)" name="bluerov2_heavy_thrusters" />
 </robot>

Commit message: ready for docs

File: blue_demos/control_integration/description/ros2_control/bluerov2.ros2_control.xacro (robot description, xacro)
@@ -44,11 +44,4 @@
       </joint>
     </ros2_control>
-    <ros2_control name="${name}_odom_sensor" type="sensor">
-      <hardware>
-        <plugin>topic_sensors/OdomSensor</plugin>
-        <param name="topic">/model/bluerov2/odometry_fsd</param>
-        <param name="prefix">${prefix}</param>
-      </hardware>
-    </ros2_control>
   </xacro:macro>
 </robot>

File: blue_demos/control_integration/description/ros2_control/bluerov2_heavy.ros2_control.xacro (robot description, xacro)
@@ -56,11 +56,4 @@
       </joint>
     </ros2_control>
-    <ros2_control name="${name}_odom_sensor" type="sensor">
-      <hardware>
-        <plugin>topic_sensors/OdomSensor</plugin>
-        <param name="topic">/model/bluerov2_heavy/odometry_fsd</param>
-        <param name="prefix">${prefix}</param>
-      </hardware>
-    </ros2_control>
   </xacro:macro>
 </robot>

File: blue_demos/control_integration/description/urdf/bluerov2_heavy.config.xacro (robot description, xacro)
@@ -4,5 +4,5 @@
   <xacro:include filename="$(find blue_description)/description/bluerov2_heavy/gazebo.xacro" />
   <xacro:include filename="$(find blue_demos)/control_integration/description/ros2_control/bluerov2_heavy.ros2_control.xacro" />
-  <xacro:include filename="$(find blue_demos)/control_integration/description/ros2_control/bluerov2.model.xacro" />
+  <xacro:include filename="$(find blue_demos)/control_integration/description/ros2_control/bluerov2_heavy.model.xacro" />
   <xacro:arg name="prefix" default="" />
   <xacro:arg name="use_sim" default="false" />

File: blue_demos/manipulator_systems/description/urdf/uvms.urdf.xacro (robot description, xacro)
@@ -17,5 +17,5 @@
         <origin rpy="0 0 0" xyz="0.11425 0.14375 0.08" />
         <geometry>
-          <box size="0.2285 0.2875 0.015" />
+          <box size="0.2285 0.2875 0.018" />
         </geometry>
       </collision>

Commit message: Added payload and integrated med manipulator demos

File: blue_demos/control_integration/description/ros2_control/bluerov2.ros2_control.xacro (robot description, xacro)
@@ -1,9 +1,10 @@
 <?xml version="1.0"?>
 <robot xmlns:xacro="http://www.ros.org/wiki/xacro">
-  <xacro:macro name="ardusub_thruster_system" params="prefix name max_set_param_attempts:=^3">
+  <xacro:macro name="ardusub_thruster_system" params="prefix name max_set_param_attempts:=^3 set_param_timeout:=^5">
     <ros2_control name="${name}" type="system">
       <hardware>
         <plugin>thruster_hardware/ThrusterHardware</plugin>
         <param name="max_set_param_attempts">${max_set_param_attempts}</param>
+        <param name="set_param_timeout">${set_param_timeout}</param>
       </hardware>
       <joint name="${prefix}thruster1_joint">

File: blue_demos/control_integration/description/ros2_control/bluerov2_heavy.ros2_control.xacro (robot description, xacro)
@@ -1,9 +1,10 @@
 <?xml version="1.0"?>
 <robot xmlns:xacro="http://www.ros.org/wiki/xacro">
-  <xacro:macro name="ardusub_thruster_system" params="prefix name max_set_param_attempts:=^3">
+  <xacro:macro name="ardusub_thruster_system" params="prefix name max_set_param_attempts:=^3 set_param_timeout:=^5">
     <ros2_control name="${name}" type="system">
       <hardware>
         <plugin>thruster_hardware/ThrusterHardware</plugin>
         <param name="max_set_param_attempts">${max_set_param_attempts}</param>
+        <param name="set_param_timeout">${set_param_timeout}</param>
       </hardware>
       <joint name="${prefix}thruster1_joint">

File: blue_demos/manipulator_systems/description/ros2_control/uvms.ros2_control.xacro (robot description, xacro)
@@ -1,7 +1,9 @@
 <?xml version="1.0"?>
 <robot xmlns:xacro="http://www.ros.org/wiki/xacro">
-  <xacro:macro name="uvms_system" params="prefix arm_prefix name initial_positions_file">
+  <xacro:macro name="uvms_system" params="prefix arm_prefix name initial_positions_file joint_limits_file">
     <xacro:property name="initial_positions_file" default="$(arg initial_positions_file)" />
     <xacro:property name="initial_positions" value="${xacro.load_yaml(initial_positions_file)['initial_positions']}" />
+    <xacro:property name="joint_limits_file" default="$(arg joint_limits_file)" />
+    <xacro:property name="joint_limits" value="${xacro.load_yaml(joint_limits_file)['joint_limits']}" />
     <ros2_control name="UVMSControlSystem" type="system">
       <hardware>
@@ -11,6 +13,6 @@
         <param name="device_id">1</param>
         <command_interface name="position">
-          <param name="min">0</param>
-          <param name="max">0.015</param>
+          <param name="min">${joint_limits['axis_a']['min_position']}</param>
+          <param name="max">${joint_limits['axis_a']['max_position']}</param>
         </command_interface>
         <command_interface name="velocity">
@@ -32,6 +34,6 @@
         <param name="device_id">2</param>
         <command_interface name="position">
-          <param name="min">0</param>
-          <param name="max">3.22</param>
+          <param name="min">${joint_limits['axis_b']['min_position']}</param>
+          <param name="max">${joint_limits['axis_b']['max_position']}</param>
         </command_interface>
         <command_interface name="velocity">
@@ -53,6 +55,6 @@
         <param name="device_id">3</param>
         <command_interface name="position">
-          <param name="min">0</param>
-          <param name="max">3.22</param>
+          <param name="min">${joint_limits['axis_c']['min_position']}</param>
+          <param name="max">${joint_limits['axis_c']['max_position']}</param>
         </command_interface>
         <command_interface name="velocity">
@@ -74,6 +76,6 @@
         <param name="device_id">4</param>
         <command_interface name="position">
-          <param name="min">0</param>
-          <param name="max">3.49</param>
+          <param name="min">${joint_limits['axis_d']['min_position']}</param>
+          <param name="max">${joint_limits['axis_d']['max_position']}</param>
         </command_interface>
         <command_interface name="velocity">
@@ -95,6 +97,6 @@
         <param name="device_id">5</param>
         <command_interface name="position">
-          <param name="min">0</param>
-          <param name="max">6.14</param>
+          <param name="min">${joint_limits['axis_e']['min_position']}</param>
+          <param name="max">${joint_limits['axis_e']['max_position']}</param>
         </command_interface>
         <command_interface name="velocity">

File: blue_demos/manipulator_systems/description/urdf/uvms.config.xacro (robot description, xacro)
@@ -9,8 +9,9 @@
   <xacro:arg name="initial_positions_file" default="$(find blue_demos)/manipulator_systems/config/initial_positions.yaml" />
   <xacro:arg name="controllers_file" default="$(find blue_demos)/manipulator_systems/config/uvms_controllers.yaml" />
-  <xacro:uvms_urdf prefix="$(arg prefix)" arm_prefix="$(arg arm_prefix)" />
+  <xacro:arg name="joint_limits_file" default="$(find blue_demos)/manipulator_systems/config/joint_limits.yaml" />
+  <xacro:uvms_urdf prefix="$(arg prefix)" arm_prefix="$(arg arm_prefix)" joint_limits_file="$(arg joint_limits_file)" />
   <xacro:uvms_gazebo prefix="$(arg prefix)" controllers_file="$(arg controllers_file)" />
   <xacro:uvms_system prefix="$(arg prefix)" arm_prefix="$(arg arm_prefix)" name="uvms_system"
-    initial_positions_file="$(arg initial_positions_file)" />
+    initial_positions_file="$(arg initial_positions_file)" joint_limits_file="$(arg joint_limits_file)" />
   <xacro:uvms_model />
 </robot>

File: blue_demos/manipulator_systems/description/urdf/uvms.urdf.xacro (robot description, xacro)
@@ -1,13 +1,19 @@
 <?xml version="1.0"?>
 <robot xmlns:xacro="http://ros.org/wiki/xacro">
-  <xacro:macro name="uvms_urdf" params="prefix arm_prefix">
-    <xacro:include filename="$(find blue_description)/description/bluerov2_heavy_reach/urdf.xacro" />
+  <xacro:macro name="uvms_urdf" params="prefix arm_prefix joint_limits_file">
+    <xacro:include filename="$(find blue_description)/description/bluerov2_heavy_reach_payload/urdf.xacro" />
     <xacro:include filename="$(find reach_description)/description/alpha_5/urdf.xacro" />
     <xacro:include filename="$(find reach_description)/description/alpha_5/standard_jaws/standard_jaws.urdf.xacro" />
     <link name="${prefix}mount_link" />
     <joint name="${prefix}mount_joint" type="fixed">
-      <origin rpy="0 0 0" xyz="0.13 -0.109 0.029" />
+      <origin rpy="0 0 0" xyz="0.093805 -0.1095 0.092075" />
       <parent link="${prefix}base_link" />
       <child link="${prefix}mount_link" />
+    </joint>
+    <link name="${prefix}connector_link" />
+    <joint name="${prefix}connector_joint" type="fixed">
+      <origin rpy="0 0 0" xyz="0.0374 0 -0.0225" />
+      <parent link="${prefix}mount_link" />
+      <child link="${prefix}connector_link" />
     </joint>
     <!-- add some additional floats to the vehicle to compensate for the manipulator -->
@@ -40,6 +46,7 @@
       <child link="${prefix}float_link" />
     </joint>
-    <xacro:bluerov2_heavy_reach_urdf prefix="${prefix}" />
-    <xacro:alpha_5_urdf parent="${prefix}mount_link" prefix="${prefix}${arm_prefix}" mount_rotation="3.14159">
+    <xacro:bluerov2_heavy_reach_payload_urdf prefix="${prefix}" />
+    <xacro:alpha_5_urdf parent="${prefix}connector_link" prefix="${prefix}${arm_prefix}"
+      joint_limits_file="${joint_limits_file}" mount_rotation="3.14159">
       <origin rpy="0 0 0" xyz="0 0 0" />
     </xacro:alpha_5_urdf>
