Commit message: Continue porting angler to demo

File: blue_demos/manipulator_systems/description/ros2_control/angler.model.xacro (robot description, xacro)
@@ -1,5 +1,5 @@
 <?xml version="1.0"?>
 <robot xmlns:xacro="http://www.ros.org/wiki/xacro">
-  <xacro:macro name="uvms_model">
+  <xacro:macro name="angler_model">
     <hydrodynamics>
       <inertial>

File: blue_demos/manipulator_systems/description/urdf/angler.urdf.xacro (robot description, xacro)
@@ -13,5 +13,4 @@
     </joint>
     <!-- add some additional floats to the vehicle to compensate for the manipulator -->
-    <!-- gazebo doesn't detect any added floats that we integrate in hardware -->
     <link name="${prefix}float_link">
       <!-- Front left -->
