Commit message: debugging alpha + bluerov integration

File: blue_demos/manipulator_systems/description/ros2_control/uvms.model.xacro (robot description, xacro)
@@ -1,5 +1,5 @@
 <?xml version="1.0"?>
 <robot xmlns:xacro="http://www.ros.org/wiki/xacro">
-  <xacro:macro name="angler_model">
+  <xacro:macro name="uvms_model">
     <hydrodynamics>
       <inertial>

File: blue_demos/manipulator_systems/description/ros2_control/uvms.ros2_control.xacro (robot description, xacro)
@@ -1,69 +1,141 @@
 <?xml version="1.0"?>
 <robot xmlns:xacro="http://www.ros.org/wiki/xacro">
-  <xacro:macro name="angler_system" params="prefix name initial_positions_file max_set_param_attempts:=^3">
-    <ros2_control name="${name}_vehicle" type="system">
+  <xacro:macro name="uvms_system" params="prefix alpha_prefix name initial_positions_file max_set_param_attempts:=^3">
+    <xacro:property name="initial_positions_file" default="$(arg initial_positions_file)" />
+    <xacro:property name="initial_positions" value="${xacro.load_yaml(initial_positions_file)['initial_positions']}" />
+    <ros2_control name="UVMS" type="system">
       <hardware>
-        <plugin>thruster_hardware/ThrusterHardware</plugin>
-        <param name="max_set_param_attempts">${max_set_param_attempts}</param>
+        <plugin>gz_ros2_control/GazeboSimSystem</plugin>
       </hardware>
       <joint name="${prefix}thruster1_joint">
-        <param name="param_name">SERVO1_FUNCTION</param>
-        <param name="default_param_value">33</param>
-        <param name="channel">1</param>
-        <command_interface name="pwm" />
+        <command_interface name="velocity" />
       </joint>
       <joint name="${prefix}thruster2_joint">
-        <param name="param_name">SERVO2_FUNCTION</param>
-        <param name="default_param_value">34</param>
-        <param name="channel">2</param>
-        <command_interface name="pwm" />
+        <command_interface name="velocity" />
       </joint>
       <joint name="${prefix}thruster3_joint">
-        <param name="param_name">SERVO3_FUNCTION</param>
-        <param name="default_param_value">35</param>
-        <param name="channel">3</param>
-        <command_interface name="pwm" />
+        <command_interface name="velocity" />
       </joint>
       <joint name="${prefix}thruster4_joint">
-        <param name="param_name">SERVO4_FUNCTION</param>
-        <param name="default_param_value">36</param>
-        <param name="channel">4</param>
-        <command_interface name="pwm" />
+        <command_interface name="velocity" />
       </joint>
       <joint name="${prefix}thruster5_joint">
-        <param name="param_name">SERVO5_FUNCTION</param>
-        <param name="default_param_value">37</param>
-        <param name="channel">5</param>
-        <command_interface name="pwm" />
+        <command_interface name="velocity" />
       </joint>
       <joint name="${prefix}thruster6_joint">
-        <param name="param_name">SERVO6_FUNCTION</param>
-        <param name="default_param_value">38</param>
-        <param name="channel">6</param>
-        <command_interface name="pwm" />
+        <command_interface name="velocity" />
       </joint>
       <joint name="${prefix}thruster7_joint">
-        <param name="param_name">SERVO7_FUNCTION</param>
-        <param name="default_param_value">39</param>
-        <param name="channel">7</param>
-        <command_interface name="pwm" />
+        <command_interface name="velocity" />
       </joint>
       <joint name="${prefix}thruster8_joint">
-        <param name="param_name">SERVO8_FUNCTION</param>
-        <param name="default_param_value">40</param>
-        <param name="channel">8</param>
-        <command_interface name="pwm" />
+        <command_interface name="velocity" />
+      </joint>
+      <joint name="${prefix}${alpha_prefix}axis_a">
+        <param name="device_id">1</param>
+        <command_interface name="position">
+          <param name="min">0</param>
+          <param name="max">0.015</param>
+        </command_interface>
+        <command_interface name="velocity">
+          <param name="min">-0.003</param>
+          <param name="max">0.003</param>
+        </command_interface>
+        <command_interface name="effort" />
+        <state_interface name="position">
+          <param name="initial_value">${initial_positions['axis_a']}</param>
+        </state_interface>
+        <state_interface name="velocity">
+          <param name="initial_value">0.0</param>
+        </state_interface>
+        <state_interface name="effort">
+          <param name="initial_value">0.0</param>
+        </state_interface>
+      </joint>
+      <joint name="${prefix}${alpha_prefix}axis_b">
+        <param name="device_id">2</param>
+        <command_interface name="position">
+          <param name="min">0</param>
+          <param name="max">3.22</param>
+        </command_interface>
+        <command_interface name="velocity">
+          <param name="min">-0.8726646</param>
+          <param name="max">0.8726646</param>
+        </command_interface>
+        <command_interface name="effort" />
+        <state_interface name="position">
+          <param name="initial_value">${initial_positions['axis_b']}</param>
+        </state_interface>
+        <state_interface name="velocity">
+          <param name="initial_value">0.0</param>
+        </state_interface>
+        <state_interface name="effort">
+          <param name="initial_value">0.0</param>
+        </state_interface>
+      </joint>
+      <joint name="${prefix}${alpha_prefix}axis_c">
+        <param name="device_id">3</param>
+        <command_interface name="position">
+          <param name="min">0</param>
+          <param name="max">3.22</param>
+        </command_interface>
+        <command_interface name="velocity">
+          <param name="min">-0.5235988</param>
+          <param name="max">0.5235988</param>
+        </command_interface>
+        <command_interface name="effort" />
+        <state_interface name="position">
+          <param name="initial_value">${initial_positions['axis_c']}</param>
+        </state_interface>
+        <state_interface name="velocity">
+          <param name="initial_value">0.0</param>
+        </state_interface>
+        <state_interface name="effort">
+          <param name="initial_value">0.0</param>
+        </state_interface>
+      </joint>
+      <joint name="${prefix}${alpha_prefix}axis_d">
+        <param name="device_id">4</param>
+        <command_interface name="position">
+          <param name="min">0</param>
+          <param name="max">3.49</param>
+        </command_interface>
+        <command_interface name="velocity">
+          <param name="min">-0.5235988</param>
+          <param name="max">0.5235988</param>
+        </command_interface>
+        <command_interface name="effort" />
+        <state_interface name="position">
+          <param name="initial_value">${initial_positions['axis_d']}</param>
+        </state_interface>
+        <state_interface name="velocity">
+          <param name="initial_value">0.0</param>
+        </state_interface>
+        <state_interface name="effort">
+          <param name="initial_value">0.0</param>
+        </state_interface>
+      </joint>
+      <joint name="${prefix}${alpha_prefix}axis_e">
+        <param name="device_id">5</param>
+        <command_interface name="position">
+          <param name="min">0</param>
+          <param name="max">6.14</param>
+        </command_interface>
+        <command_interface name="velocity">
+          <param name="min">-0.5235988</param>
+          <param name="max">0.5235988</param>
+        </command_interface>
+        <command_interface name="effort" />
+        <state_interface name="position">
+          <param name="initial_value">${initial_positions['axis_e']}</param>
+        </state_interface>
+        <state_interface name="velocity">
+          <param name="initial_value">0.0</param>
+        </state_interface>
+        <state_interface name="effort">
+          <param name="initial_value">0.0</param>
+        </state_interface>
       </joint>
     </ros2_control>
-    <ros2_control name="${name}_odom_sensor" type="sensor">
-      <hardware>
-        <plugin>topic_sensors/OdomSensor</plugin>
-        <param name="topic">/model/angler/odometry_fsd</param>
-        <param name="prefix">${prefix}</param>
-      </hardware>
-    </ros2_control>
-    <xacro:include filename="$(find reach_description)/description/alpha_5/ros2_control.xacro" />
-    <xacro:alpha_5_system prefix="${prefix}alpha_" initial_positions_file="$(arg initial_positions_file)" use_sim="true"
-      use_mock_hardware="false" serial_port="" />
   </xacro:macro>
 </robot>

File: blue_demos/manipulator_systems/description/urdf/uvms.config.xacro (robot description, xacro)
@@ -1,4 +1,4 @@
 <?xml version="1.0"?>
-<robot name="angler" xmlns:xacro="http://ros.org/wiki/xacro">
+<robot name="uvms" xmlns:xacro="http://ros.org/wiki/xacro">
   <xacro:include filename="$(find blue_demos)/manipulator_systems/description/urdf/uvms.urdf.xacro" />
   <xacro:include filename="$(find blue_demos)/manipulator_systems/description/urdf/uvms.gazebo.xacro" />
@@ -8,7 +8,7 @@
   <xacro:arg name="initial_positions_file" default="$(find blue_demos)/manipulator_systems/config/initial_positions.yaml" />
   <xacro:arg name="controllers_file" default="$(find blue_demos)/manipulator_systems/config/uvms_controllers.yaml" />
-  <xacro:angler_urdf prefix="$(arg prefix)" />
-  <xacro:angler_gazebo prefix="$(arg prefix)" controllers_file="$(arg controllers_file)" />
-  <xacro:angler_model />
-  <xacro:angler_system prefix="$(arg prefix)" name="angler_system" initial_positions_file="$(arg initial_positions_file)" />
+  <xacro:uvms_urdf prefix="$(arg prefix)" />
+  <xacro:uvms_gazebo prefix="$(arg prefix)" controllers_file="$(arg controllers_file)" />
+  <xacro:uvms_model />
+  <xacro:uvms_system prefix="$(arg prefix)" name="uvms_system" initial_positions_file="$(arg initial_positions_file)" />
 </robot>

File: blue_demos/manipulator_systems/description/urdf/uvms.gazebo.xacro (robot description, xacro)
@@ -1,9 +1,12 @@
 <?xml version="1.0"?>
 <robot xmlns:xacro="http://ros.org/wiki/xacro">
-  <xacro:macro name="angler_gazebo" params="prefix controllers_file">
-    <xacro:include filename="$(find blue_description)/description/bluerov2_heavy_reach/gazebo.xacro" />
-    <xacro:include filename="$(find reach_description)/description/alpha_5/gz.xacro" />
-    <xacro:bluerov2_heavy_reach_gazebo prefix="${prefix}" />
-    <xacro:alpha_5_gazebo prefix="${prefix}" controllers_file="${controllers_file}" />
+  <xacro:macro name="uvms_gazebo" params="prefix controllers_file">
+    <gazebo>
+      <plugin filename="gz_ros2_control-system"
+        name="gz_ros2_control::GazeboSimROS2ControlPlugin">
+        <parameters>${controllers_file}</parameters>
+      </plugin>
+    </gazebo>
+    <!-- TODO(evan-palmer): port bluerov2 gazebo stuff to here -->
   </xacro:macro>
 </robot>

File: blue_demos/manipulator_systems/description/urdf/uvms.urdf.xacro (robot description, xacro)
@@ -1,9 +1,8 @@
 <?xml version="1.0"?>
 <robot xmlns:xacro="http://ros.org/wiki/xacro">
-  <xacro:macro name="angler_urdf" params="prefix">
+  <xacro:macro name="uvms_urdf" params="prefix">
     <xacro:include filename="$(find blue_description)/description/bluerov2_heavy_reach/urdf.xacro" />
     <xacro:include filename="$(find reach_description)/description/alpha_5/urdf.xacro" />
     <xacro:include filename="$(find reach_description)/description/alpha_5/standard_jaws/standard_jaws.urdf.xacro" />
-    <!-- create a mount for the manipulator -->
     <link name="${prefix}mount_link" />
     <joint name="${prefix}mount_joint" type="fixed">
@@ -41,7 +40,5 @@
       <child link="${prefix}float_link" />
     </joint>
-    <!-- BlueROV2 -->
     <xacro:bluerov2_heavy_reach_urdf prefix="${prefix}" />
-    <!-- Alpha 5 -->
     <xacro:alpha_5_urdf parent="${prefix}mount_link" prefix="${prefix}alpha_" mount_rotation="3.14159">
       <origin rpy="0 0 0" xyz="0 0 0" />
