Commit message: Fixed arm mount

File: blue_demos/manipulator_systems/description/ros2_control/uvms.ros2_control.xacro (robot description, xacro)
@@ -1,5 +1,5 @@
 <?xml version="1.0"?>
 <robot xmlns:xacro="http://www.ros.org/wiki/xacro">
-  <xacro:macro name="angler_system" params="prefix name init_positions_file max_set_param_attempts:=^3">
+  <xacro:macro name="angler_system" params="prefix name initial_positions_file max_set_param_attempts:=^3">
     <ros2_control name="${name}_vehicle" type="system">
       <hardware>
@@ -63,7 +63,7 @@
       </hardware>
     </ros2_control>
-    <xacro:include filename="$(find reach_description)/description/alpha_5/ros2_control.xacro" />
-    <xacro:alpha_5_system prefix="${prefix}" initial_positions_file="$(arg init_positions_file)" use_sim="true"
-      use_mock_hardware="false" />
+    <!-- <xacro:include filename="$(find reach_description)/description/alpha_5/ros2_control.xacro" /> -->
+    <!-- <xacro:alpha_5_system prefix="${prefix}" initial_positions_file="$(arg initial_positions_file)" use_sim="true"
+      use_mock_hardware="false" serial_port="" /> -->
   </xacro:macro>
 </robot>

File: blue_demos/manipulator_systems/description/urdf/uvms.gazebo.xacro (robot description, xacro)
@@ -5,5 +5,5 @@
     <xacro:include filename="$(find reach_description)/description/alpha_5/gz.xacro" />
     <xacro:bluerov2_heavy_reach_gazebo prefix="${prefix}" />
-    <xacro:alpha_5_gazebo prefix="${prefix}" controllers_file="${controllers_file}" />
+    <!-- <xacro:alpha_5_gazebo prefix="${prefix}" controllers_file="${controllers_file}" /> -->
   </xacro:macro>
 </robot>

File: blue_demos/manipulator_systems/description/urdf/uvms.urdf.xacro (robot description, xacro)
@@ -8,5 +8,5 @@
     <link name="${prefix}mount_link" />
     <joint name="${prefix}mount_joint" type="fixed">
-      <origin rpy="0 0 0" xyz="0.24 -0.099 0.029" />
+      <origin rpy="0 0 0" xyz="0.13 -0.109 0.029" />
       <parent link="${prefix}base_link" />
       <child link="${prefix}mount_link" />
@@ -37,6 +37,6 @@
     </link>
     <joint name="${prefix}float_joint" type="fixed">
-      <xacro:insert_block name="origin" />
-      <parent link="${parent}" />
+      <origin rpy="0 0 0" xyz="0 0 0" />
+      <parent link="${prefix}base_link" />
       <child link="${prefix}float_link" />
     </joint>
@@ -44,8 +44,8 @@
     <xacro:bluerov2_heavy_reach_urdf prefix="${prefix}" />
     <!-- Alpha 5 -->
-    <xacro:alpha_5_urdf parent="${prefix}mount_link" prefix="${prefix}alpha_">
-      <origin xyz="0 0 0" rpy="0 0 0" />
+    <xacro:alpha_5_urdf parent="${prefix}mount_link" prefix="${prefix}alpha_" mount_rotation="3.14159">
+      <origin rpy="0 0 0" xyz="0 0 0" />
     </xacro:alpha_5_urdf>
-    <xacro:standard_jaws parent="${prefix}rs1_124_link" prefix="${prefix}alpha_" mimic_joint="${prefix}axis_a" />
+    <xacro:standard_jaws parent="${prefix}alpha_rs1_124_link" prefix="${prefix}alpha_" mimic_joint="${prefix}alpha_axis_a" />
   </xacro:macro>
 </robot>

Commit message: base launch for uvms demo working

File: blue_demos/manipulator_systems/description/ros2_control/uvms.ros2_control.xacro (robot description, xacro)
@@ -1,5 +1,5 @@
 <?xml version="1.0"?>
 <robot xmlns:xacro="http://www.ros.org/wiki/xacro">
-  <xacro:macro name="uvms_system" params="prefix alpha_prefix name initial_positions_file max_set_param_attempts:=^3">
+  <xacro:macro name="uvms_system" params="prefix arm_prefix name initial_positions_file max_set_param_attempts:=^3">
     <xacro:property name="initial_positions_file" default="$(arg initial_positions_file)" />
     <xacro:property name="initial_positions" value="${xacro.load_yaml(initial_positions_file)['initial_positions']}" />
@@ -32,5 +32,5 @@
         <command_interface name="velocity" />
       </joint>
-      <joint name="${prefix}${alpha_prefix}axis_a">
+      <joint name="${prefix}${arm_prefix}axis_a">
         <param name="device_id">1</param>
         <command_interface name="position">
@@ -53,5 +53,5 @@
         </state_interface>
       </joint>
-      <joint name="${prefix}${alpha_prefix}axis_b">
+      <joint name="${prefix}${arm_prefix}axis_b">
         <param name="device_id">2</param>
         <command_interface name="position">
@@ -74,5 +74,5 @@
         </state_interface>
       </joint>
-      <joint name="${prefix}${alpha_prefix}axis_c">
+      <joint name="${prefix}${arm_prefix}axis_c">
         <param name="device_id">3</param>
         <command_interface name="position">
@@ -95,5 +95,5 @@
         </state_interface>
       </joint>
-      <joint name="${prefix}${alpha_prefix}axis_d">
+      <joint name="${prefix}${arm_prefix}axis_d">
         <param name="device_id">4</param>
         <command_interface name="position">
@@ -116,5 +116,5 @@
         </state_interface>
       </joint>
-      <joint name="${prefix}${alpha_prefix}axis_e">
+      <joint name="${prefix}${arm_prefix}axis_e">
         <param name="device_id">5</param>
         <command_interface name="position">

File: blue_demos/manipulator_systems/description/urdf/uvms.config.xacro (robot description, xacro)
@@ -6,9 +6,11 @@
   <xacro:include filename="$(find blue_demos)/manipulator_systems/description/ros2_control/uvms.model.xacro" />
   <xacro:arg name="prefix" default="" />
+  <xacro:arg name="arm_prefix" default="alpha_" />
   <xacro:arg name="initial_positions_file" default="$(find blue_demos)/manipulator_systems/config/initial_positions.yaml" />
   <xacro:arg name="controllers_file" default="$(find blue_demos)/manipulator_systems/config/uvms_controllers.yaml" />
-  <xacro:uvms_urdf prefix="$(arg prefix)" />
+  <xacro:uvms_urdf prefix="$(arg prefix)" arm_prefix="$(arg arm_prefix)" />
   <xacro:uvms_gazebo prefix="$(arg prefix)" controllers_file="$(arg controllers_file)" />
+  <xacro:uvms_system prefix="$(arg prefix)" arm_prefix="$(arg arm_prefix)" name="uvms_system"
+    initial_positions_file="$(arg initial_positions_file)" />
   <xacro:uvms_model />
-  <xacro:uvms_system prefix="$(arg prefix)" name="uvms_system" initial_positions_file="$(arg initial_positions_file)" />
 </robot>

File: blue_demos/manipulator_systems/description/urdf/uvms.gazebo.xacro (robot description, xacro)
@@ -8,5 +8,42 @@
       </plugin>
     </gazebo>
-    <!-- TODO(evan-palmer): port bluerov2 gazebo stuff to here -->
+    <gazebo>
+      <plugin filename="gz-sim-hydrodynamics-system" name="gz::sim::systems::Hydrodynamics">
+        <link_name>${prefix}base_footprint</link_name>
+        <!-- Added mass -->
+        <xDotU>0</xDotU>
+        <yDotV>0</yDotV>
+        <zDotW>0</zDotW>
+        <kDotP>0</kDotP>
+        <mDotQ>0</mDotQ>
+        <nDotR>0</nDotR>
+        <!-- First order stability derivative -->
+        <xU>0</xU>
+        <yV>0</yV>
+        <zW>0</zW>
+        <kP>0</kP>
+        <mQ>0</mQ>
+        <nR>0</nR>
+        <!-- Second order stability derivative -->
+        <xUabsU>-58.42</xUabsU>
+        <yVabsV>-55.137</yVabsV>
+        <zWabsW>-124.818</zWabsW>
+        <kPabsP>-4.0</kPabsP>
+        <mQabsQ>-4.0</mQabsQ>
+        <nRabsR>-4.0</nRabsR>
+      </plugin>
+    </gazebo>
+    <gazebo>
+      <plugin
+        filename="gz-sim-odometry-publisher-system"
+        name="gz::sim::systems::OdometryPublisher">
+        <odom_frame>map</odom_frame>
+        <robot_base_frame>${prefix}base_link</robot_base_frame>
+        <dimensions>3</dimensions>
+        <odom_publish_frequency>100</odom_publish_frequency>
+      </plugin>
+    </gazebo>
+    <xacro:include filename="$(find blue_description)/description/camera/gazebo.xacro" />
+    <xacro:camera_gazebo reference="${prefix}camera_mount_link" />
   </xacro:macro>
 </robot>

File: blue_demos/manipulator_systems/description/urdf/uvms.urdf.xacro (robot description, xacro)
@@ -1,5 +1,5 @@
 <?xml version="1.0"?>
 <robot xmlns:xacro="http://ros.org/wiki/xacro">
-  <xacro:macro name="uvms_urdf" params="prefix">
+  <xacro:macro name="uvms_urdf" params="prefix arm_prefix">
     <xacro:include filename="$(find blue_description)/description/bluerov2_heavy_reach/urdf.xacro" />
     <xacro:include filename="$(find reach_description)/description/alpha_5/urdf.xacro" />
@@ -41,8 +41,9 @@
     </joint>
     <xacro:bluerov2_heavy_reach_urdf prefix="${prefix}" />
-    <xacro:alpha_5_urdf parent="${prefix}mount_link" prefix="${prefix}alpha_" mount_rotation="3.14159">
+    <xacro:alpha_5_urdf parent="${prefix}mount_link" prefix="${prefix}${arm_prefix}" mount_rotation="3.14159">
       <origin rpy="0 0 0" xyz="0 0 0" />
     </xacro:alpha_5_urdf>
-    <xacro:standard_jaws parent="${prefix}alpha_rs1_124_link" prefix="${prefix}alpha_" mimic_joint="${prefix}alpha_axis_a" />
+    <xacro:standard_jaws parent="${prefix}${arm_prefix}rs1_124_link" prefix="${prefix}${arm_prefix}"
+      mimic_joint="${prefix}${arm_prefix}axis_a" />
   </xacro:macro>
 </robot>

Commit message: controllers integrated need to test tpik control

File: blue_demos/manipulator_systems/description/ros2_control/uvms.ros2_control.xacro (robot description, xacro)
@@ -1,5 +1,5 @@
 <?xml version="1.0"?>
 <robot xmlns:xacro="http://www.ros.org/wiki/xacro">
-  <xacro:macro name="uvms_system" params="prefix arm_prefix name initial_positions_file max_set_param_attempts:=^3">
+  <xacro:macro name="uvms_system" params="prefix arm_prefix name initial_positions_file">
     <xacro:property name="initial_positions_file" default="$(arg initial_positions_file)" />
     <xacro:property name="initial_positions" value="${xacro.load_yaml(initial_positions_file)['initial_positions']}" />
@@ -8,28 +8,4 @@
         <plugin>gz_ros2_control/GazeboSimSystem</plugin>
       </hardware>
-      <joint name="${prefix}thruster1_joint">
-        <command_interface name="velocity" />
-      </joint>
-      <joint name="${prefix}thruster2_joint">
-        <command_interface name="velocity" />
-      </joint>
-      <joint name="${prefix}thruster3_joint">
-        <command_interface name="velocity" />
-      </joint>
-      <joint name="${prefix}thruster4_joint">
-        <command_interface name="velocity" />
-      </joint>
-      <joint name="${prefix}thruster5_joint">
-        <command_interface name="velocity" />
-      </joint>
-      <joint name="${prefix}thruster6_joint">
-        <command_interface name="velocity" />
-      </joint>
-      <joint name="${prefix}thruster7_joint">
-        <command_interface name="velocity" />
-      </joint>
-      <joint name="${prefix}thruster8_joint">
-        <command_interface name="velocity" />
-      </joint>
       <joint name="${prefix}${arm_prefix}axis_a">
         <param name="device_id">1</param>

File: blue_demos/manipulator_systems/description/urdf/uvms.gazebo.xacro (robot description, xacro)
@@ -44,4 +44,13 @@
       </plugin>
     </gazebo>
+    <xacro:include filename="$(find blue_description)/description/t200/gazebo.xacro" />
+    <xacro:t200_gazebo namespace="uvms" prefix="${prefix}" id="1" ccw="true" />
+    <xacro:t200_gazebo namespace="uvms" prefix="${prefix}" id="2" ccw="true" />
+    <xacro:t200_gazebo namespace="uvms" prefix="${prefix}" id="3" />
+    <xacro:t200_gazebo namespace="uvms" prefix="${prefix}" id="4" />
+    <xacro:t200_gazebo namespace="uvms" prefix="${prefix}" id="5" ccw="true" />
+    <xacro:t200_gazebo namespace="uvms" prefix="${prefix}" id="6" />
+    <xacro:t200_gazebo namespace="uvms" prefix="${prefix}" id="7" />
+    <xacro:t200_gazebo namespace="uvms" prefix="${prefix}" id="8" ccw="true" />
   </xacro:macro>
 </robot>
